Commit message: Added tool obj and modified urdf

File: 04-mmp_panda/mmp_panda_tool_collision.urdf (robot description, URDF)
Before this commit: robot mmp_panda, 12 links, 11 joints
Links:
- link base_link: geometry collision mesh filename=../../../models/mmp_panda/meshes/panda_BaseCombo.obj; visual mesh filename=../../../models/mmp_panda/meshes/panda_BaseCombo.obj
- link link1: geometry collision mesh filename=../../../models/panda/meshes/collision/link1.obj; visual mesh filename=../../../models/panda/meshes/visual/link1.obj
- link link2: geometry collision mesh filename=../../../models/panda/meshes/collision/link2.obj; visual mesh filename=../../../models/panda/meshes/visual/link2.obj
- link link3: geometry collision mesh filename=../../../models/panda/meshes/collision/link3.obj; visual mesh filename=../../../models/panda/meshes/visual/link3.obj
- link link4: geometry collision mesh filename=../../../models/panda/meshes/collision/link4.obj; visual mesh filename=../../../models/panda/meshes/visual/link4.obj
- link link5: geometry collision mesh filename=../../../models/panda/meshes/collision/link5.obj; visual mesh filename=../../../models/panda/meshes/visual/link5.obj
- link link6: geometry collision mesh filename=../../../models/panda/meshes/collision/link6.obj; visual mesh filename=../../../models/panda/meshes/visual/link6.obj
- link link7: geometry collision mesh filename=../../../models/panda/meshes/collision/link7.obj; visual mesh filename=../../../models/panda/meshes/visual/link7.obj
- link linkTool: geometry collision mesh filename=../../../models/Drill2/Drill2.obj; visual mesh filename=../../../models/Drill2/Drill2.obj
