Commit message: 04-mmp_panda/ and construction/ work independently

File: 04-mmp_panda/mmp_panda.urdf (robot description, URDF)
Before this commit: robot mmp_panda, 12 links, 11 joints
Links:
- link base_link: geometry visual mesh filename=../../../model/mmp_panda/meshes/panda_BaseCombo.obj
- link link1: geometry visual mesh filename=../../../model/panda/meshes/visual/link1.obj
- link link2: geometry visual mesh filename=../../../model/panda/meshes/visual/link2.obj
- link link3: geometry visual mesh filename=../../../model/panda/meshes/visual/link3.obj
- link link4: geometry visual mesh filename=../../../model/panda/meshes/visual/link4.obj
- link link5: geometry visual mesh filename=../../../model/panda/meshes/visual/link5.obj
- link link6: geometry visual mesh filename=../../../model/panda/meshes/visual/link6.obj
- link link7: geometry visual mesh filename=../../../model/panda/meshes/visual/link7.obj
- link linkTool: geometry visual mesh filename=../../../model/Drill2/Drill2.obj

File: 04-mmp_panda/mmp_panda_tool_collision.urdf (robot description, URDF)
Before this commit: robot mmp_panda, 12 links, 11 joints
Links:
- link base_link: geometry collision mesh filename=../../../model/mmp_panda/meshes/panda_BaseCombo.obj; visual mesh filename=../../../model/mmp_panda/meshes/panda_BaseCombo.obj
- link link1: geometry collision mesh filename=../../../model/panda/meshes/collision/link1.obj; visual mesh filename=../../../model/panda/meshes/visual/link1.obj
- link link2: geometry collision mesh filename=../../../model/panda/meshes/collision/link2.obj; visual mesh filename=../../../model/panda/meshes/visual/link2.obj
- link link3: geometry collision mesh filename=../../../model/panda/meshes/collision/link3.obj; visual mesh filename=../../../model/panda/meshes/visual/link3.obj
- link link4: geometry collision mesh filename=../../../model/panda/meshes/collision/link4.obj; visual mesh filename=../../../model/panda/meshes/visual/link4.obj
- link link5: geometry collision mesh filename=../../../model/panda/meshes/collision/link5.obj; visual mesh filename=../../../model/panda/meshes/visual/link5.obj
- link link6: geometry collision mesh filename=../../../model/panda/meshes/collision/link6.obj; visual mesh filename=../../../model/panda/meshes/visual/link6.obj
- link link7: geometry collision mesh filename=../../../model/panda/meshes/collision/link7.obj; visual mesh filename=../../../model/panda/meshes/visual/link7.obj
- link linkTool: geometry collision mesh filename=../../../model/Drill2/Drill2.obj; visual mesh filename=../../../model/Drill2/Drill2.obj

File: 04-mmp_panda/mmp_panda_tool_no_collision.urdf (robot description, URDF)
Before this commit: robot mmp_panda, 12 links, 11 joints
Links:
- link base_link: geometry visual mesh filename=../../../model/mmp_panda/meshes/panda_BaseCombo.obj
- link link1: geometry visual mesh filename=../../../model/panda/meshes/visual/link1.obj
- link link2: geometry visual mesh filename=../../../model/panda/meshes/visual/link2.obj
- link link3: geometry visual mesh filename=../../../model/panda/meshes/visual/link3.obj
- link link4: geometry visual mesh filename=../../../model/panda/meshes/visual/link4.obj
- link link5: geometry visual mesh filename=../../../model/panda/meshes/visual/link5.obj
- link link6: geometry visual mesh filename=../../../model/panda/meshes/visual/link6.obj
- link link7: geometry visual mesh filename=../../../model/panda/meshes/visual/link7.obj
- link linkTool: geometry visual mesh filename=../../../model/Drill2/Drill2.obj

File: construction/mmp_panda.urdf (robot description, URDF)
Before this commit: robot mmp_panda, 11 links, 10 joints
Links:
- added link linkTool, mass 1; visual mesh filename=../../../model/Drill2/Drill2.obj
Joints:
- added joint jointTool: type fixed, parent link7, child linkTool, origin xyz=0 0 0.107 rpy=0 3.14159265359 0, axis 0 0 1, limit lower=-2.8973 upper=2.8973 effort=12 velocity=2.6100

File: construction/mmp_panda_tool_collision.urdf (robot description, URDF)
Before this commit: robot mmp_panda, 12 links, 11 joints
Links:
- link base_link: geometry collision mesh filename=../../../model/mmp_panda/meshes/panda_BaseCombo.obj; visual mesh filename=../../../model/mmp_panda/meshes/panda_BaseCombo.obj
- link link1: geometry collision mesh filename=../../../model/panda/meshes/collision/link1.obj; visual mesh filename=../../../model/panda/meshes/visual/link1.obj
- link link2: geometry collision mesh filename=../../../model/panda/meshes/collision/link2.obj; visual mesh filename=../../../model/panda/meshes/visual/link2.obj
- link link3: geometry collision mesh filename=../../../model/panda/meshes/collision/link3.obj; visual mesh filename=../../../model/panda/meshes/visual/link3.obj
- link link4: geometry collision mesh filename=../../../model/panda/meshes/collision/link4.obj; visual mesh filename=../../../model/panda/meshes/visual/link4.obj
- link link5: geometry collision mesh filename=../../../model/panda/meshes/collision/link5.obj; visual mesh filename=../../../model/panda/meshes/visual/link5.obj
- link link6: geometry collision mesh filename=../../../model/panda/meshes/collision/link6.obj; visual mesh filename=../../../model/panda/meshes/visual/link6.obj
- link link7: geometry collision mesh filename=../../../model/panda/meshes/collision/link7.obj; visual mesh filename=../../../model/panda/meshes/visual/link7.obj
- link linkTool: geometry collision mesh filename=../../../model/Drill2/Drill2.obj; visual mesh filename=../../../model/Drill2/Drill2.obj

Commit message: Added tall base obj

File: 04-mmp_panda/mmp_panda.urdf (robot description, URDF)
Before this commit: robot mmp_panda, 12 links, 11 joints
Links:
- added link base_z, mass 0.001
- link base_link: geometry visual mesh filename=../../../models/mmp_panda_tall/meshes/panda_TallBaseCombo.o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
Joints:
- added joint base_prismatic_z: type prismatic, parent base_y, child base_z, origin xyz=0 0 0 rpy=0 0 0, axis 0 0 1, limit lower=-2.8973 upper=2.9873 effort=87 velocity=2.1750
- joint base_revolute: parent base_y -> base_z
