Commit message: slimmed 04-mmp_panda, only use files in construction/ directory

File: construction/mmp_panda.urdf (robot description, URDF)
Before this commit: robot mmp_panda, 12 links, 11 joints
Links:
- added link base_z, mass 0.001
- link base_link: geometry visual mesh filename=../../../model/mmp_panda_tall/meshes/panda_TallBaseCombo.obj
Joints:
- added joint base_prismatic_z: type prismatic, parent base_y, child base_z, origin xyz=0 0 0 rpy=0 0 0, axis 0 0 1, limit lower=-2.8973 upper=2.9873 effort=87 velocity=2.1750
- joint base_revolute: parent base_y -> base_z

Commit message: initial position and limits matching gui

File: construction/mmp_panda.urdf (robot description, URDF)
Before this commit: robot mmp_panda, 13 links, 12 joints
Joints:
- joint base_prismatic_x: limit lower=-2.8973 upper=2.9873 effort=87 velocity=2.1750 -> lower=-5 upper=5. effort=87 velocity=0.2
- joint base_prismatic_y: limit lower=-2.8973 upper=2.9873 effort=87 velocity=2.1750 -> lower=-5 upper=5 effort=87 velocity=0.2
- joint base_prismatic_z: limit lower=-2.8973 upper=2.9873 effort=87 velocity=2.1750 -> lower=-1.0 upper=2.0 effort=87 velocity=0.2
- joint jointTool: limit lower=-2.8973 upper=2.8973 effort=12 velocity=2.6100 -> (none)

Commit message: adjusted mmp_panda.urdf  to match updated tool orientation

File: construction/mmp_panda.urdf (robot description, URDF)
Before this commit: robot mmp_panda, 13 links, 12 joints
Joints:
- joint jointTool: origin xyz=0 0 0.107 rpy=0 3.14159265359 0 -> xyz=0 0 0.104 rpy=0 0 0

Commit message: made more realistic base, modified urdf and gui html

File: construction/mmp_panda.urdf (robot description, URDF)
Before this commit: robot mmp_panda, 13 links, 12 joints
Links:
- removed link base_link
- added link base_fix, mass 0.001
- added link base_theta, mass 2230; visual mesh filename=../../../model/mmp_panda_tall/meshes/WideBase.obj
- link base_z: mass 0.001 -> 64.6; geometry visual mesh filename=../../../model/mmp_panda_tall/meshes/panda_TallBaseCombo.obj
- link linkTool: mass 1 -> 2.2
Joints:
- added joint base_fixed: type fixed, parent base_theta, child base_fix, origin xyz=0 0 0 rpy=0 0 0, axis 0 0 1, limit lower=0 upper=2.0 effort=87 velocity=0.2
- joint base_prismatic_x: limit lower=-5 upper=5. effort=87 velocity=0.2 -> lower=-5 upper=5 effort=87 velocity=0.2
- joint base_prismatic_z: limit lower=-1.0 upper=2.0 effort=87 velocity=0.2 -> lower=0 upper=2.0 effort=87 velocity=0.2; parent base_y -> base_fix
- joint base_revolute: child base_link -> base_theta; parent base_z -> base_y
- joint joint1: parent base_link -> base_z

Commit message: cylinder radius and length changed

File: construction/mmp_panda.urdf (robot description, URDF)
Before this commit: robot mmp_panda, 14 links, 13 joints
Links:
- link linkTool: geometry collision cylinder length=0.203 radius=0.104; visual mesh filename=../../../model/Drill2/Drill2.obj

Commit message: corrected base orientataion in urdf

File: construction/mmp_panda.urdf (robot description, URDF)
Before this commit: robot mmp_panda, 14 links, 13 joints
Links:
- link base_theta: mass 2230 -> 64.6
Joints:
- joint base_fixed: origin xyz=0 0 0 rpy=0 0 0 -> xyz=0 0 0 rpy=0 0 1.57079632679

Commit message: updated inertia in mmp_panda.urdf

File: construction/mmp_panda.urdf (robot description, URDF)
Before this commit: robot mmp_panda, 14 links, 13 joints
Links:
- link base_theta: mass 64.6 -> 2230
- link linkTool: geometry collision cylinder length=0.25 radius=0.05; visual mesh filename=../../../model/Drill2/Drill2.obj

Commit message: new drill w/o bolt added

File: construction/mmp_panda.urdf (robot description, URDF)
Before this commit: robot mmp_panda, 14 links, 13 joints
Links:
- link linkTool: geometry visual mesh filename=../../../model/Drill_NoBolt/drill_nobolt.obj

Commit message: adjusted base color

File: construction/mmp_panda.urdf (robot description, URDF)
Before this commit: robot mmp_panda, 14 links, 13 joints
Links:
- link linkTool: geometry visual mesh filename=../../../model/Drill2/Drill2.obj
